Commit message: Update code release

File: urdf/thesis_robot_new.xacro (robot description, xacro)
@@ -172,12 +172,13 @@
   </joint>
   <link name="imu_link"/>
+ <!-- Lidar -->
   <joint name="scan_joint" type="fixed">
     <parent link="base_link"/>
     <child link="base_scan"/>
-    <origin xyz="0 0 0.175" rpy="0 0 3.14159"/>
+    <origin xyz="0 0 0.175" rpy="0 0 0"/>
   </joint>
   <link name="base_scan">
     <visual>
-      <origin xyz="0 0 0.0" rpy="0 0 3.14159"/>
+      <origin xyz="0 0 0.0" rpy="0 0 0"/>
       <geometry>
         <mesh filename="package://thesis_robot_new/urdf/lds.stl" scale="0.001 0.001 0.001"/>
